Commit message: Migrate EVA-H1 robot description to Xacro

File: src/eva_h1_description/urdf/eva_h1.urdf.xacro (robot description, xacro)
@@ -1,4 +1,5 @@
 <?xml version="1.0"?>
-<robot name="eva_h1">
+<robot xmlns:xacro="http://www.ros.org/wiki/xacro"
+       name="eva_h1">
   <link name="base_link">
     <visual>
@@ -242,8 +243,10 @@
 </inertial>
 </link>
-<joint name="left_wheel_joint" type="fixed">
+<joint name="left_wheel_joint" type="continuous">
   <parent link="left_axle_link"/>
   <child link="left_wheel_link"/>
-  <origin xyz="0.07 0 -0.05" rpy="0 1.5708 0"/>
+  <origin xyz="0.07 0 -0.05"
+          rpy="0 1.5708 0"/>
+  <axis xyz="0 1 0"/>
 </joint>
 <link name="right_axle_link">
@@ -298,8 +301,17 @@
 </inertial>
 </link>
-<joint name="right_wheel_joint" type="fixed">
+<joint name="right_wheel_joint" type="continuous">
   <parent link="right_axle_link"/>
   <child link="right_wheel_link"/>
-  <origin xyz="-0.07 0 -0.05" rpy="0 1.5708 0"/>
-</joint>
+  <origin xyz="-0.07 0 -0.05"
+          rpy="0 1.5708 0"/>
+  <axis xyz="0 1 0"/>
+</joint>
+<gazebo>
+  <plugin
+      name="gazebo_ros2_control"
+      filename="libgazebo_ros2_control.so">
+    <parameters>$(find eva_h1_description)/config/controllers.yaml</parameters>
+  </plugin>
+</gazebo>S
 </robot>

Commit message: Integrate ros2_control with wheel velocity controllers

File: src/eva_h1_description/urdf/eva_h1.urdf.xacro (robot description, xacro)
@@ -308,4 +308,19 @@
   <axis xyz="0 1 0"/>
 </joint>
+<ros2_control name="EvaH1System" type="system">
+  <hardware>
+    <plugin>gazebo_ros2_control/GazeboSystem</plugin>
+  </hardware>
+  <joint name="left_wheel_joint">
+    <command_interface name="velocity"/>
+    <state_interface name="position"/>
+    <state_interface name="velocity"/>
+  </joint>
+  <joint name="right_wheel_joint">
+    <command_interface name="velocity"/>
+    <state_interface name="position"/>
+    <state_interface name="velocity"/>
+  </joint>
+</ros2_control>
 <gazebo>
   <plugin
